Commit message: update training 10k

File: oped_description/urdf/leg.urdf.xacro (robot description, xacro)
@@ -150,5 +150,5 @@
             <axis xyz="0 1 0" />
             <!-- <limit effort="1000" lower="-${pi}" upper="${pi}" velocity="1.5" /> -->
-            <limit effort="1000" lower="-1.5" upper="1.5" velocity="1.5" />
+            <limit effort="1000" lower="-2" upper="2" velocity="1.5" />
             <!-- <limit effort="1000" lower="-0.68" upper="0.68" velocity="1.5" /> -->
             <parent link="${leg}_hip_link" />
@@ -164,17 +164,17 @@
             <child link="${leg}_lower_leg_link" />
             <xacro:if value="${leg == 'lf'}">
-                <limit effort="1000" lower="-1.8" upper="0.5" velocity="1.5" />
+                <limit effort="1000" lower="-3" upper="0.5" velocity="1.5" />
                 <origin xyz="0 0.0015 -${upper_leg_to_lower_leg_distance}" rpy="0 0 0" />
             </xacro:if>
             <xacro:if value="${leg == 'lh'}">
-                <limit effort="1000" lower="-0.5" upper="1.8" velocity="1.5" />
+                <limit effort="1000" lower="-0.5" upper="3" velocity="1.5" />
                 <origin xyz="0 0.0015 -${upper_leg_to_lower_leg_distance}" rpy="0 0 0" />
             </xacro:if>
             <xacro:if value="${leg == 'rf'}">
-                <limit effort="1000" lower="-1.8" upper="0.5" velocity="1.5" />
+                <limit effort="1000" lower="-3" upper="0.5" velocity="1.5" />
                 <origin xyz="0 -0.002 -${upper_leg_to_lower_leg_distance}" rpy="0 0 0" />
             </xacro:if>
             <xacro:if value="${leg == 'rh'}">
-                <limit effort="1000" lower="-0.5" upper="1.8" velocity="1.5" />
+                <limit effort="1000" lower="-0.5" upper="3" velocity="1.5" />
                 <origin xyz="0 -0.002 -${upper_leg_to_lower_leg_distance}" rpy="0 0 0" />
             </xacro:if>

File: oped_description/urdf/oped.urdf (robot description, URDF)
Before this commit: robot oped, 23 links, 22 joints
Joints:
- joint lf_lower_leg_joint: limit lower=-1.8 upper=0.5 effort=1000 velocity=1.5 -> lower=-3 upper=0.5 effort=1000 velocity=1.5
- joint lf_upper_leg_joint: limit lower=-1.5 upper=1.5 effort=1000 velocity=1.5 -> lower=-2 upper=2 effort=1000 velocity=1.5
- joint lh_lower_leg_joint: limit lower=-0.5 upper=1.8 effort=1000 velocity=1.5 -> lower=-0.5 upper=3 effort=1000 velocity=1.5
- joint lh_upper_leg_joint: limit lower=-1.5 upper=1.5 effort=1000 velocity=1.5 -> lower=-2 upper=2 effort=1000 velocity=1.5
- joint rf_lower_leg_joint: limit lower=-1.8 upper=0.5 effort=1000 velocity=1.5 -> lower=-3 upper=0.5 effort=1000 velocity=1.5
- joint rf_upper_leg_joint: limit lower=-1.5 upper=1.5 effort=1000 velocity=1.5 -> lower=-2 upper=2 effort=1000 velocity=1.5
- joint rh_lower_leg_joint: limit lower=-0.5 upper=1.8 effort=1000 velocity=1.5 -> lower=-0.5 upper=3 effort=1000 velocity=1.5
- joint rh_upper_leg_joint: limit lower=-1.5 upper=1.5 effort=1000 velocity=1.5 -> lower=-2 upper=2 effort=1000 velocity=1.5
